File: schematic/Vacuum2/Vacuum2.kicad_sch (KiCad schematic)
At the start: 4 parts, among them M1 Motor_DC, M2 Motor_DC, U1 STM32F411CEUx, U2 TB6612FNG

Commit message: update schematic
Parts:
- added PROG, RESET: SW_Push, symbol Switch:SW_Push
- added R1: R, symbol Device:R
- added U3: ESP32-WROOM-32, RF_Module:ESP32-WROOM-32, symbol RF_Module:ESP32-WROOM-32
- added U4: MCP1825S, symbol Regulator_Linear:MCP1825S
Connections:
- net GND: now also PROG.2, RESET.1, U3.1 (GND), U3.15 (GND), U3.38 (GND), U3.39 (GND), U4.2 (GND)
- net DATA_READY: now reaches U1.11 (PA1)
- net DATA_READY: now also U3.27 (IO16)
- net SPI_CS: now reaches U1.25 (PB12)
- net SPI_CS: now also U3.23 (IO15)
- net SCLK: now reaches U1.26 (PB13)
- net SCLK: now also U3.13 (IO14)
- net MISO: now reaches U1.27 (PB14)
- net MISO: now also U3.14 (IO12)
- net MOSI: now reaches U1.28 (PB15)
- net MOSI: now also U3.16 (IO13)
- new net: PROG.1, U3.25 (IO0)
- new net: R1.2, U3.3 (EN)
- new net +3V3: R1.1, RESET.2, U3.2 (VDD), U4.3 (VO)
- new net +5V: U4.1 (VI)
